File: cap_pcb.kicad_sch (KiCad schematic)
At the start: 10 parts, among them J1 Conn_02x09_Odd_Even, J14 PL Pins, J2 Conn_02x09_Odd_Even, J3 Conn_02x09_Odd_Even, J4 Conn_02x09_Odd_Even, J5 Conn_02x09_Odd_Even, J6 Conn_02x09_Odd_Even, J7 Conn_02x09_Odd_Even, J8 Conn_02x09_Odd_Even, J9 Conn_02x09_Odd_Even

Commit message: - Added capacitors on HDMI TDMS lines
Parts:
- added C1: 47uf 25v, Capacitor_SMD:C_1206_3216Metric, symbol Device:C
- added C10, C11, C12, C5, C6, C7, C8, C9: 100n, Capacitor_SMD:C_0603_1608Metric_Pad1.08x0.95mm_HandSolder, symbol Device:C_Small
- added C2: 100 uf 10v, Capacitor_SMD:C_1206_3216Metric, symbol Device:C
- added C3: 100n, Capacitor_SMD:C_1206_3216Metric, symbol Device:C
- added C4: 1n, Capacitor_SMD:C_1206_3216Metric, symbol Device:C
- added J10: USB Expansion board, Connector_PinSocket_2.54mm:PinSocket_2x10_P2.54mm_Horizontal, symbol Connector_Generic:Conn_02x10_Odd_Even
- added J11: Aux_mio_conn, Connector_PinHeader_2.54mm:PinHeader_1x05_P2.54mm_Vertical, symbol Connector:Conn_01x05_Pin
- added J12: 12v Pwr, Connector_PinSocket_2.54mm:PinSocket_2x02_P2.54mm_Vertical, symbol Connector_Generic:Conn_02x02_Odd_Even
- added J13: HDMI_A, Connector_Video:HDMI_A_Molex_208658-1001_Horizontal, symbol Connector:HDMI_A
- added R1: 1m, Resistor_SMD:R_1206_3216Metric, symbol Device:R
- added RN1, RN2: TC164-FR-0749R9L, SamacSys_Parts:TC164FR0749R9L, symbol SamacSys_Parts:TC164-FR-0749R9L
- added TP1: CEC, TestPoint:TestPoint_Pad_D2.0mm, symbol Connector:TestPoint
- added TP2: SCL, TestPoint:TestPoint_Pad_D2.0mm, symbol Connector:TestPoint
- added TP3: SDA, TestPoint:TestPoint_Pad_D2.0mm, symbol Connector:TestPoint
- added TP4: HPD, TestPoint:TestPoint_Pad_D2.0mm, symbol Connector:TestPoint
- added TP5: UTILITY, TestPoint:TestPoint_Pad_D2.0mm, symbol Connector:TestPoint
- added TP6: 5V_HDMI, TestPoint:TestPoint_Pad_D2.0mm, symbol Connector:TestPoint
- added U1: L7805, Package_TO_SOT_THT:TO-220-3_Horizontal_TabDown, symbol Regulator_Linear:L7805
Connections:
- net 3.3V: now also J10.19 (Pin_19), J10.20 (Pin_20), RN1.5, RN1.6, RN1.7, RN1.8, RN2.5, RN2.6, RN2.7, RN2.8; no longer J2.16 (Pin_16)
- net BANK34_L11N_RST6: now also C12.1
- net BANK34_L11P_PLUG6: now also C11.1
- net BANK34_L12N_RXD6: now also C10.1
- net BANK34_L12P_TXD6: now also C9.1
- net BANK34_L15N_RST7: now also C8.1
- net BANK34_L15P__PLUG7: now also C7.1
- net BANK34_L16N_RXD7: now also C6.1
- net BANK34_L16P_TXD7: now also C5.1
- net GND: now also C1.2, C2.2, C3.2, C4.2, J10.17 (Pin_17), J10.18 (Pin_18), J12.2 (Pin_2), J12.4 (Pin_4), J13.11 (CKS), J13.17 (GND), J13.2 (D2S), J13.5 (D1S), J13.8 (D0S), R1.2, U1.2 (GND)
- net PS_MIO30: now also J10.16 (Pin_16)
- net PS_MIO28 renamed DATA4
- net DATA4: now also J10.9 (Pin_9)
- net PS_MIO29 renamed DIR
- net DIR: now also J10.12 (Pin_12)
- net PS_MIO31 renamed NXT
- net NXT: now also J10.14 (Pin_14)
- net PS_MIO32 renamed DATA0
- net DATA0: now also J10.1 (Pin_1)
- net PS_MIO33 renamed DATA1
- net DATA1: now also J10.3 (Pin_3)
- net PS_MIO34 renamed DATA2
- net DATA2: now also J10.5 (Pin_5)
- net PS_MIO35 renamed DATA3
- net DATA3: now also J10.7 (Pin_7)
- net PS_MIO36 renamed CLK
- net CLK: now also J10.10 (Pin_10)
- new net: J13.15 (SCL), TP2.1
- new net: C8.2, J13.6 (D1-), RN1.4
- new net: C7.2, J13.4 (D1+), RN1.3
- new net: J13.18 (+5V), TP6.1
- new net: C4.1, J13.SH, R1.1
- new net: C5.2, J13.1 (D2+), RN1.1
- new net: C11.2, J13.10 (CK+), RN2.2
- new net: C12.2, J13.12 (CK-), RN2.1
- new net: J13.13 (CEC), TP1.1
- new net: J13.14 (UTILITY), TP5.1
- new net: J13.16 (SDA), TP3.1
- new net: J13.19 (HPD), TP4.1
- new net: C6.2, J13.3 (D2-), RN1.2
- new net: C9.2, J13.7 (D0+), RN2.4
- new net: C10.2, J13.9 (D0-), RN2.3
- new net +12V: C1.1, J12.1 (Pin_1), J12.3 (Pin_3), U1.1 (IN)
- new net +5V: C2.1, C3.1, J10.2 (Pin_2), J10.4 (Pin_4), U1.3 (OUT)
- new net 2.5VCC_IO: J10.6 (Pin_6), J11.5 (Pin_5)
- new net DATA5: J10.11 (Pin_11), J11.1 (Pin_1)
- new net DATA6: J10.13 (Pin_13), J11.2 (Pin_2)
- new net DATA7: J10.15 (Pin_15), J11.3 (Pin_3)
- new net RST: J10.8 (Pin_8), J11.4 (Pin_4)
Other:
- note added: "Usb to Zynq mapping"
- moved on the sheet: J5, J6, J7, J8, J9
