File: hdmi.kicad_sch (KiCad schematic)
At the start: 5 parts, among them J13 HDMI_A

Commit message: - Added capacitors on HDMI TDMS lines
Parts:
- removed C4: 1n, Capacitor_SMD:C_1206_3216Metric, symbol Device:C
- removed J13: HDMI_A, Connector_Video:HDMI_A_Molex_208658-1001_Horizontal, symbol Connector:HDMI_A
- removed R1: 1m, Resistor_SMD:R_1206_3216Metric, symbol Device:R
- removed RN1, RN2: TC164-FR-0749R9L, SamacSys_Parts:TC164FR0749R9L, symbol SamacSys_Parts:TC164-FR-0749R9L
