File: modules.kicad_sch (KiCad schematic)
At the start: 19 parts, among them J15 Conn_02x06 Extension, J16 Conn_01x02_Pin, J17 SD_MODULE_CONN, J18 EMMC_CONN, U3 TPS5430DDA

Commit message: Updates for version 1.1:  - Project named as Antminer_hat_pcb  - Added USB3315 Phy on board  - Removed ULPI connector  - Optimized HDMI wiring  - Other updates
Parts:
- removed C15, C16, C17: 22uf 25v, Capacitor_SMD:C_1206_3216Metric, symbol Device:C
- removed C18: 10n, Capacitor_SMD:C_1206_3216Metric_Pad1.33x1.80mm_HandSolder, symbol Device:C
- removed C19: 10uf 50v, Capacitor_SMD:C_1206_3216Metric_Pad1.33x1.80mm_HandSolder, symbol Device:C
- removed C20, C21, C22: 47uf 10v, Capacitor_Tantalum_SMD:CP_EIA-3528-12_Kemet-T, symbol Device:C
- removed D3: SS54, Diode_SMD:D_SMC_Handsoldering, symbol Diode:SS34
- removed D5: WS2812B-B/T, LED_SMD:LED_WS2812B_PLCC4_5.0x5.0mm_P3.2mm, symbol LED:WS2812B
- removed J15: Conn_02x06 Extension, Connector_PinHeader_1.27mm:PinHeader_2x06_P1.27mm_Vertical, symbol Connector_Generic:Conn_02x06_Counter_Clockwise
- removed J16: Conn_01x02_Pin, Connector_PinHeader_2.54mm:PinHeader_1x02_P2.54mm_Vertical, symbol Connector:Conn_01x02_Pin
- removed J17: SD_MODULE_CONN, Connector_PinHeader_2.54mm:PinHeader_2x10_P2.54mm_Vertical, symbol Connector_Generic:Conn_02x10_Odd_Even
- removed J18: EMMC_CONN, Connector_PinHeader_1.27mm:PinHeader_2x10_P1.27mm_Vertical_SMD, symbol Connector_Generic:Conn_02x10_Odd_Even
- removed L3: 22uh 4A, Inductor_SMD:L_Sunlord_MWSA1003S, symbol Device:L
- removed R7: 10k, Resistor_SMD:R_1206_3216Metric, symbol Device:R
- removed R8: 3k3, Resistor_SMD:R_1206_3216Metric, symbol Device:R
- removed R9: 150k, Resistor_SMD:R_1206_3216Metric, symbol Device:R
- removed U3: TPS5430DDA, Package_SO:TI_SO-PowerPAD-8_ThermalVias, symbol Regulator_Switching:TPS5430DDA
Other:
- note removed: "AUX module"
- note removed: "EMMC module"
