File: usb_conn.kicad_sch (KiCad schematic)
At the start: 7 parts, among them J10 USB Expansion board, J11 Aux_mio_conn, J12 12v Pwr, U1 L7805

Commit message: - Added capacitors on HDMI TDMS lines
Parts:
- removed C1: 47uf 25v, Capacitor_SMD:C_1206_3216Metric, symbol Device:C
- removed C2: 100 uf 10v, Capacitor_SMD:C_1206_3216Metric, symbol Device:C
- removed C3: 100n, Capacitor_SMD:C_1206_3216Metric, symbol Device:C
- removed J10: USB Expansion board, Connector_PinSocket_2.54mm:PinSocket_2x10_P2.54mm_Horizontal, symbol Connector_Generic:Conn_02x10_Odd_Even
- removed J11: Aux_mio_conn, Connector_PinHeader_2.54mm:PinHeader_1x05_P2.54mm_Vertical, symbol Connector:Conn_01x05_Pin
- removed J12: 12v Pwr, Connector_PinSocket_2.54mm:PinSocket_2x02_P2.54mm_Vertical, symbol Connector_Generic:Conn_02x02_Odd_Even
- removed U1: L7805, Package_TO_SOT_THT:TO-220-3_Horizontal_TabDown, symbol Regulator_Linear:L7805
Other:
- note removed: "Usb to Zynq mapping"

Commit message: Updates for version 1.1:  - Project named as Antminer_hat_pcb  - Added USB3315 Phy on board  - Removed ULPI connector  - Optimized HDMI wiring  - Other updates
Parts:
- added C13, C23, C25, C5, C6: 0.1uf, Capacitor_SMD:C_0805_2012Metric, symbol Device:C_Small
- added C14, C24: 10uf, Capacitor_SMD:C_1206_3216Metric_Pad1.33x1.80mm_HandSolder, symbol Device:C_Small
- added C7: 100uf, Capacitor_SMD:C_1210_3225Metric_Pad1.33x2.70mm_HandSolder, symbol Device:C_Small
- added C8: 1n, Capacitor_SMD:C_1206_3216Metric_Pad1.33x1.80mm_HandSolder, symbol Device:C_Small
- added D1: CDDFN10-0524P, SamacSys_Parts:CDDFN100524P, symbol SamacSys_Parts:CDDFN10-0524P
- added D2, D8: LED, LED_SMD:LED_1210_3225Metric_Pad1.42x2.65mm_HandSolder, symbol Device:LED
- added D4: 1N5822, Diode_SMD:D_1206_3216Metric_Pad1.42x1.75mm_HandSolder, symbol Diode:1N5822
- added IC1: USB3315C-CP-TR, QFN50P400X400X100-25N-D, symbol SamacSys_Parts:USB3315C-CP-TR
- added IC2: LM3525M-H, SamacSys_Parts:SOIC127P620X175-8N, symbol SamacSys_Parts:LM3525M-H
- added J14: USB_C_Receptacle_USB2.0_16P, Connector_USB:USB_C_Receptacle_GCT_USB4105-xx-A_16P_TopMnt_Horizontal, symbol Connector:USB_C_Receptacle_USB2.0_16P
- added J15: 48204-0001 China, 482040001, symbol SamacSys_Parts:48204-0001
- added R10, R11, R12, R13, R14, R15, R16, R17, R18, R19, R6: 30, Resistor_SMD:R_0805_2012Metric, symbol Device:R_Small
- added R2: 820, Resistor_SMD:R_0805_2012Metric, symbol Device:R_Small
- added R20, R3: 2k, Resistor_SMD:R_0805_2012Metric, symbol Device:R_Small
- added R21: 1M, Resistor_SMD:R_0805_2012Metric, symbol Device:R_Small
- added R4: 4k7, Resistor_SMD:R_0805_2012Metric, symbol Device:R_Small
- added R5: 8k06, Resistor_SMD:R_0805_2012Metric, symbol Device:R_Small
- added U2: LM1117DT-1.8, Package_TO_SOT_SMD:SOT-223-3_TabPin2, symbol Regulator_Linear:LM1117DT-1.8
- added Y1: 24Mhz, Oscillator:Oscillator_SMD_Abracon_ASV-4Pin_7.0x5.1mm, symbol Oscillator:ASV-xxxMHz
Connections:
- new net: D1.1 (LINE_-1), D1.10 (NC_4), D1.2 (LINE-2), D1.9 (NC_3), IC1.1 (ID), J14.A5 (CC1), J14.B5 (CC2)
- new net: IC1.10 (DATA5), R11.1
- new net: IC1.11 (DATA4), R10.1
- new net: IC1.12 (CLKOUT), R6.1
- new net: IC1.13 (DATA3), R14.1
- new net: IC1.14 (DATA2), R15.1
- new net: IC1.15 (DATA1), R16.1
- new net: IC1.16 (DATA0), R17.1
- new net: IC1.18 (NXT), R18.1
- new net: IC1.19 (DIR), R19.1
- new net: IC1.2 (VBUS), R2.2
- new net: IC1.23 (REFCLK), Y1.3 (OUT)
- new net: IC1.24 (RBIAS), R5.2
- new net: IC1.7 (CPEN), IC2.1 (EN)
- new net: IC1.8 (DATA7), R13.1
- new net: IC1.9 (DATA6), R12.1
- new net: D2.1 (K), R3.2
- new net: C8.1, J14.S1 (SHIELD), J15.5 (Shield), J15.6 (Shield), J15.7 (Shield), J15.8 (Shield), R21.2
- new net: IC2.2 (FLAG), R3.1
- new net: D8.2 (A), R20.2
- new net: R4.1, Y1.1 (EN)
- new net +1.8V: C23.1, C24.1, IC1.21 (VDD1.8), U2.2 (VO)
- new net +3.3V: C13.1, C14.1, C25.1, IC1.3 (VBAT), IC1.4 (VDD3.3), R4.2, Y1.4 (Vdd)
- new net +5V: D2.2 (A), D4.1 (K), IC2.7 (IN), U2.3 (VI)
- new net 2.5VCC_IO: C5.1, IC1.17 (VDDIO)
- new net CLK: R6.2
- new net DATA0: R17.2
- new net DATA1: R16.2
- new net DATA2: R15.2
- new net DATA3: R14.2
- new net DATA4: R10.2
- new net DATA5: R11.2
- new net DATA6: R12.2
- new net DATA7: R13.2
- new net DIR: R19.2
- new net GND: C13.2, C14.2, C23.2, C24.2, C25.2, C5.2, C6.2, C7.2, C8.2, D1.3 (GND), D8.1 (K), IC1.25 (GND), IC2.3 (GND), J14.A1 (GND), J14.A12 (GND), J14.B1 (GND), J14.B12 (GND), J15.1 (GND), R21.1, R5.1, U2.1 (GND), Y1.2 (GND)
- new net NXT: R18.2
- new net RST: IC1.22 (RESETB)
- new net STP: IC1.20 (STP)
- new net USB_D+: D1.5 (LINE-4), D1.6 (NC_1), IC1.6 (DP), J14.A6 (D+), J14.B6 (D+), J15.2 (D+)
- new net USB_D-: D1.4 (LINE-3), D1.7 (NC_2), IC1.5 (DM), J14.A7 (D-), J14.B7 (D-), J15.3 (D-)
- new net V_BUS: C6.1, C7.1, D4.2 (A), IC2.6 (OUT_2), IC2.8 (OUT), J14.A4 (VBUS), J14.A9 (VBUS), J14.B4 (VBUS), J14.B9 (VBUS), J15.4 (V_BUS), R2.1, R20.1
Other:
- title: (none) -> KCC Tech hat board for Antminer S9
